File: clock-to-midi.kicad_sch (KiCad schematic)
At the start: 10 parts

Commit message: refactor
Parts:
- R?: value 12k -> 120k
- R?: value 10k -> 100k
Other:
- note added: "protect against overvoltage and reverse polarity"
Changed lines of the file:
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@@
     (stroke (width 0) (type default) (color 0 0 0 0))
+  )
+  (text "protect against overvoltage\nand reverse polarity" (at 86.995 62.865 0)
+    (effects (font (size 1.27 1.27)) (justify left bottom))
   )
   (symbol (lib_id "Device:R") (at 89.535 109.855 0) (unit 1)
@@
   (symbol (lib_id "Device:R") (at 97.79 78.105 0) (unit 1)
     (in_bom yes) (on_board yes) (fields_autoplaced)
-    (property "Reference" "R?" (id 0) (at 99.695 76.8349 0)
-      (effects (font (size 1.27 1.27)) (justify left))
-    )
-    (property "Value" "12k" (id 1) (at 99.695 79.3749 0)
+    (property "Reference" "R?" (id 0) (at 100.33 76.8349 0)
+      (effects (font (size 1.27 1.27)) (justify left))
+    )
+    (property "Value" "120k" (id 1) (at 100.33 79.3749 0)
       (effects (font (size 1.27 1.27)) (justify left))
     )
@@
       (effects (font (size 1.27 1.27)) (justify left))
     )
-    (property "Value" "10k" (id 1) (at 100.33 90.8049 0)
+    (property "Value" "100k" (id 1) (at 100.33 90.8049 0)
       (effects (font (size 1.27 1.27)) (justify left))
     )
@@
     )
     (path "/da44fce3-90f3-4070-b586-dd3ea38f2708"
-      (reference "R?") (unit 1) (value "12k") (footprint "")
+      (reference "R?") (unit 1) (value "120k") (footprint "")
     )
     (path "/f4255b72-3d51-41f4-a3d5-e58520dfed20"
-      (reference "R?") (unit 1) (value "10k") (footprint "")
+      (reference "R?") (unit 1) (value "100k") (footprint "")
     )
     (path "/4eb4e693-4e46-4e15-a215-70c5cf9e7dab"

Commit message: made protoboard
Parts:
- added D2: 1N4148, kicad-official/Diode_THT.pretty:D_A-405_P2.54mm_Vertical_AnodeUp, symbol Diode:1N4148
- added J3: MIDI_IN, alchy/spacestudio_components.pretty:DIN_5, symbol Connector:DIN-5_180degree
- added R6, R7: 220, kicad-official/Resistor_THT.pretty:R_Axial_DIN0204_L3.6mm_D1.6mm_P2.54mm_Vertical, symbol Device:R
- added U2: PC817, kicad-official/Package_DIP.pretty:DIP-4_W7.62mm, symbol Isolator:PC817
- D1: renamed from D?; footprint Diode_THT:D_DO-35_SOD27_P7.62mm_Horizontal -> kicad-official/Diode_THT.pretty:D_A-405_P2.54mm_Vertical_AnodeUp
- J1: renamed from J?; value AudioJack2_Ground -> CLOCK_IN; footprint (none) -> nebs/eurocad/Eurocad.pretty:PJ301M-12
- J2: renamed from J?; value DIN-5_180degree -> MIDI_OUT; footprint (none) -> alchy/spacestudio_components.pretty:DIN_5
- R1, R2, R3, R4, R5: renamed from R?; footprint (none) -> kicad-official/Resistor_THT.pretty:R_Axial_DIN0204_L3.6mm_D1.6mm_P2.54mm_Vertical
- SW1: renamed from SW?; value SW_Push -> SW_STARTSTOP; footprint (none) -> kicad-official/Button_Switch_THT.pretty:SW_PUSH_6mm
- U1: renamed from U?; footprint (none) -> XenGi/teensy.pretty:Teensy2.0
Connections:
- net +5V: now also R7.1
- net GND: now also U1.1 (GND), U2.3; no longer U1.15 (GND)
- net at U1.9 (7_INT2_RX): now also R7.2, U2.4
- new net: D2.1 (K), R6.1, U2.1
- new net: D2.2 (A), J3.5, U2.2
- new net: J3.4, R6.2
- no-connect marks 2 -> 5
Other:
- note added: "[Optional]: pass additional singals through to out"
- note added: "https://learn.sparkfun.com/tutorials/midi-tutorial/hardware--electronic-implementation"
